File: KiCAD_Camsat_PCB/KiCAD_Camsat_PCB.kicad_sch (KiCad schematic)
At the start: 49 parts, among them J1 QWIIC_RIGHT_ANGLE, J2 QWIIC_RIGHT_ANGLE, K1 HYC77-TF09-200, K2 HEADER_MALE_6X1, Q3 BSS138, Q4 BSS138, U1 ISM330DHCX, U2 BME280, U2 MIC5225-3.3, U3 SE5218, U4 TXB0104QPWRQ1, U5 DHT11, U6 ESP32-WROOM-32E

Commit message: Payload pcb updates
Parts:
- removed J1, J2: QWIIC_RIGHT_ANGLE, KiCAD_Camsat_PCB:JST04_1MM_RA, symbol KiCAD_Camsat_PCB-eagle-import:QWIIC_CONNECTORJS-1MM
- removed JP2: HEADER-1X770MIL, KiCAD_Camsat_PCB:1X07_ROUND_70, symbol KiCAD_Camsat_PCB-eagle-import:microbuilder_HEADER-1X770MIL
- removed JP2, JP3: IO, KiCAD_Camsat_PCB:1X06_NO_SILK, symbol KiCAD_Camsat_PCB-eagle-import:CONN_06NO_SILK_NO_POP
- removed U6: ESP32-WROOM-32E, RF_Module:ESP32-WROOM-32D, symbol RF_Module:ESP32-WROOM-32E
- added C10: 10uF, symbol CL05A106MP5NUNC_C315248
- added C10: 22uF, symbol CL21A226MAYNNNE
- added C11: 4.7uF, symbol CL05A475KP5NRNC
- added C11: 100nF, symbol CL05B104KO5NNNC_1
- added C12: 10uF, symbol CL05A106MP5NUNC_C315248_1
- added C12: 100nF, symbol CL05B104KO5NNNC_5
- added C13: 100nF, symbol CL05B104KO5NNNC_3
- added C13: 100nF, symbol CL05B104KO5NNNC_2
- added C14: 100nF, symbol CL05B104KO5NNNC_7
- added C8: 100nF, symbol CL05B104KO5NNNC_4
- added C8: 100nF, symbol CL05B104KO5NNNC_6
- added C9: 100nF, symbol CL05B104KO5NNNC_8
- added C9: 100nF, symbol CL05B104KO5NNNC
- added D3: LESD5D5.0CT1G, symbol LESD5D5.0CT1G
- added D3: LESD5D5.0CT1G, symbol LESD5D5.0CT1G_2
- added D4: LESD5D5.0CT1G, symbol LESD5D5.0CT1G_1
- added J3: 105017-0001, symbol 105017-0001
- added J3: X6511WV-17H-C30D60, symbol X6511WV-17H-C30D60
- added J4: X6511WV-17H-C30D60, symbol X6511WV-17H-C30D60_1
- added J4: 210-1S-1*3Ppin Gold-plated, symbol 210-1S-1*3Ppin Gold-plated
- added J5: DZ127R-11-02-25, symbol DZ127R-11-02-25
- added LED1: 0805G (Green), symbol 0805G (Green)
- added LED2: FC-2012HRK-620D, symbol FC-2012HRK-620D
- added Q1: 2N7002T-7-F, symbol 2N7002T-7-F
- added Q1: 2N7002T-7-F, symbol 2N7002T-7-F_1
- added Q2: SS8050-G_C164885, symbol SS8050-G_C164885
- added Q2: SS8050-G_C164885, symbol SS8050-G_C164885_1
- added R11: 1kΩ, symbol 0402WGF1001TCE_1
- added R11: 47.5kΩ, symbol 0402WGF4752TCE
- added R12: 22.1kΩ, symbol 0402WGF2212TCE
- added R12: 10kΩ, symbol 0402WGF1002TCE_4
- added R13: 10kΩ, symbol 0402WGF1002TCE_2
- added R13: 10kΩ, symbol 0402WGF1002TCE_3
- added R14: 1kΩ, symbol 0402WGF1001TCE
- added R14: 22Ω, symbol 0402WGF220JTCE
- added R15: 22Ω, symbol 0402WGF220JTCE_1
- added R15: 5.1kΩ, symbol 0402WGF5101TCE
- added R16: 560Ω, symbol 0402WGF5600TCE
- added R17: 10kΩ, symbol 0402WGF1002TCE
- added R18: 10kΩ, symbol 0402WGF1002TCE_1
- added R19: 0Ω, symbol 0402WGF0000TCE
- added R20: 0Ω, symbol 0402WGF0000TCE_1
- added SW1: PTS645SH50SMTR92LFS, symbol PTS645SH50SMTR92LFS
- added SW2: PTS645SH50SMTR92LFS, symbol PTS645SH50SMTR92LFS_1
- added U7: AMS1117-3.3_C347222, symbol AMS1117-3.3_C347222
- added U8: ESP32-WROOM-32E(8MB), symbol ESP32-WROOM-32E(8MB)
- added U9: CP2102N-A02-GQFN28R, symbol CP2102N-A02-GQFN28R
Connections:
- net SCL is gone; now on net IO22: R2.1, U1.P13 (SCL)
- net SDI/SDA_5V is gone; now on net IO21: Q4.3 (D), R8.1
- net GND: now also C10.2, C10.2, C11.1, C11.1, C12.1, C12.2, C13.1, C13.1, C14.1, C8.1, C8.1, C9.1, C9.1, D3.1, D3.1, D4.1, J3.1, J3.10 (EP), J3.15, J3.5 (GND), J3.6 (EP), J3.7 (EP), J3.8 (EP), J3.9 (EP), J4.2, J4.8, LED1.2 (K), Q1.2 (S), Q1.2 (S), R11.1, R12.2, R13.1, SW1.3, SW1.4, SW2.3, SW2.4, U7.1 (ADJ(GND)), U8.1 (GND), U8.15 (GND), U8.38 (GND), U8.39 (GND), U9.29 (EP), U9.3 (GND)
- net SCLK_H: now also J4.10, LED2.1 (-), U8.30 (IO18)
- net SCK/SCL_5V renamed IO22
- net IO22: now also J4.4, U8.36 (IO22)
- net SDA/PICO renamed IO21
- net IO21: now also J4.7, U8.33 (IO21)
- new net: C9.2, J5.2, Q1.1 (G), Q1.1 (G), R11.1, R12.1
- new net: R13.2, U9.11 (SUSPENDb)
- new net: R11.2, R12.1, U9.8 (VBUS)
- new net: R14.1, U9.9 (RSTb)
- new net: LED2.2 (+), R16.1
- new net: LED1.1 (A), R15.1
- new net: Q2.1 (B), R17.2
- new net: Q2.1 (B), R18.2
- new net +3V3: C10.1, C11.2, C11.2, C12.1, C13.2, C14.2, C8.2, J3.2, J4.1, J5.1, R13.1, R14.2, R15.2, R16.2, U7.2 (VOUT(TAB)), U7.4 (TAB), U8.2 (3V3), U9.6 (VDD), U9.7 (VREGIN)
- new net +5V: C10.1, J4.2, U7.3 (VIN)
- new net +5V_EXT: C12.2, J3.17, J4.3
- new net +5V_VBUS: C8.2, D3.2, J3.1 (VCC), J4.1, R12.2
- new net DTR: Q2.2 (E), R17.1, U9.28 (DTR)
- new net EN: C9.2, J3.3, Q2.3 (C), R13.2, SW1.1, SW1.2, U8.3 (EN)
- new net I34: J3.6, U8.6 (IO34)
- new net I35: J3.7, U8.7 (IO35)
- new net I36: J3.4, U8.4 (SENSOR_VP)
- new net I39: J3.5, U8.5 (SENSOR_VN)
- new net IO0: R14.1, R15.1, U8.25 (IO0)
- new net IO0_BTN: C13.2, Q2.3 (C), R15.2, SW2.1, SW2.2
- new net IO0_CON: J4.15, R14.2
- new net IO12: J3.14, U8.14 (IO12)
- new net IO13: J3.16, U8.16 (IO13)
- new net IO14: J3.13, U8.13 (IO14)
- new net IO15: J4.17, U8.23 (IO15)
- new net IO16: J4.13, U8.27 (IO16)
- new net IO17: J4.12, U8.28 (IO17)
- new net IO19: J4.9, U8.31 (IO19)
- new net IO2: J4.16, U8.24 (IO2)
- new net IO23: J4.3, R11.2, U8.37 (IO23)
- new net IO25: J3.10, U8.10 (IO25)
- new net IO26: J3.11, U8.11 (IO26)
- new net IO27: J3.12, U8.12 (IO27)
- new net IO32: J3.8, U8.8 (IO32)
- new net IO33: J3.9, U8.9 (IO33)
- new net IO4: J4.14, U8.26 (IO4)
- new net IO5: J4.11, U8.29 (IO5)
- new net RTS: Q2.2 (E), R18.1, U9.24 (RTS)
- new net RXD: R19.2, U9.25 (RXD)
- new net RXD0: J4.6, R20.1, U8.34 (RXD0)
- new net TXD: R20.2, U9.26 (TXD)
- new net TXD0: J4.5, R19.1, U8.35 (TXD0)
- new net USB_DN: D4.2, J3.2 (D-), Q1.3 (D), U9.5 (D-)
- new net USB_DP: D3.2, J3.3 (D+), Q1.3 (D), U9.4 (D+)
- no-connect marks 0 -> 24
Other:
- note added: "5V to 3.3V"
- note added: "BOOT/USER BUTTON"
- note added: "CONNECTORS"
- note added: "ESP32 MODULE"
- note added: "NF"
- note added: "POWER INPUT SELECTION"
- note added: "POWER LED"
- note added: "RESET BUTTON"
- note added: "SDA = GPIO21 SCL = GPIO22"
- note added: "SERIAL SIGNALS HANDLING"
- note added: "These pin connections can be removed?"
- note added: "USB CONNECTOR"
- note added: "USB TO UART"
- note added: "USER LED"

Commit message: Schematic updates
Parts:
- removed C12: 100nF, symbol CL05B104KO5NNNC_5
- removed C14: 100nF, symbol CL05B104KO5NNNC_7
- removed C8: 100nF, symbol CL05B104KO5NNNC_6
- removed J3: X6511WV-17H-C30D60, symbol X6511WV-17H-C30D60
- removed J4: X6511WV-17H-C30D60, symbol X6511WV-17H-C30D60_1
- removed K2: HEADER_MALE_6X1, e-radionica.com footprinti:HEADER_MALE_6X1, symbol e-radionica.com schematics:HEADER_MALE_6X1
Connections:
- net IO19 is gone; now on net MISO_H: U8.31 (IO19)
- net IO23 is gone; now on net MOSI_H: R11.2, U8.37 (IO23)
- net IO4 is gone; now on net Signal data DT11: U8.26 (IO4)
- net IO5 is gone; now on net CS_H: U8.29 (IO5)
Other:
- note added: "SDA = GPIO21 SCL = GPIO22 CS = GPIO5 MOSI = GPIO23 SCLK = GPIO18 MISO = GPIO19"
- note removed: "CONNECTORS"
- note removed: "Connectors"
- note removed: "HEADER"
- note removed: "SDA = GPIO21 SCL = GPIO22"
- note removed: "These pin connections can be removed?"
- moved on the sheet: ADDR0, C1, C10, C11, C12, C13, C2, C3, C4, C5, C6, C7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

Commit message: 9V connector
Parts:
- added C14, C15: 470uF, Capacitor_SMD:C_0603_1608Metric, symbol CL05B104KO5NNNC
- added D5: 1N5819, Diode_THT:D_DO-41_SOD81_P10.16mm_Horizontal, symbol Diode:1N5819
- added J1: Barrel_Jack, symbol Connector:Barrel_Jack
- added L1: 33uH, symbol Device:L
- added U6: LM2596S-5, Package_TO_SOT_SMD:TO-263-5_TabPin3, symbol Regulator_Switching:LM2596S-5
- C10, C11, C12: footprint (none) -> Capacitor_SMD:C_0805_2012Metric
- C13, C8, C9: footprint (none) -> Capacitor_SMD:C_0603_1608Metric
- C16: renamed from C11; footprint (none) -> Capacitor_SMD:C_0603_1608Metric
- C17: renamed from C10; footprint (none) -> Capacitor_SMD:C_1206_3216Metric
- C20: renamed from C13; footprint (none) -> Capacitor_SMD:C_0603_1608Metric
- C25: renamed from C9; footprint (none) -> Capacitor_SMD:C_0603_1608Metric
- D3, D4: footprint (none) -> Diode_SMD:D_SOD-523
- D9: renamed from D3; footprint (none) -> Diode_SMD:D_SOD-523
- J3: footprint (none) -> Connector_USB:USB_Micro-B_Molex-105017-0001
- J4: footprint (none) -> Connector_PinHeader_2.54mm:PinHeader_1x03_P2.54mm_Vertical
- J5: footprint (none) -> Connector_PinHeader_1.27mm:PinHeader_1x02_P1.27mm_Vertical
- LED1, LED2: footprint (none) -> LED_SMD:LED_0805_2012Metric
- Q1: footprint (none) -> Package_TO_SOT_SMD:SOT-523
- Q2: footprint (none) -> Package_TO_SOT_SMD:SOT-23
- Q8: renamed from Q1; footprint (none) -> Package_TO_SOT_SMD:SOT-523
- Q9: renamed from Q2; footprint (none) -> Package_TO_SOT_SMD:SOT-23
- R10, R11, R12, R13, R14, R15, R16, R17, R18, R19, R20: footprint (none) -> Resistor_SMD:R_0805_2012Metric
- R21: renamed from R12; footprint (none) -> Resistor_SMD:R_0805_2012Metric
- R22: renamed from R13; footprint (none) -> Resistor_SMD:R_0805_2012Metric
- R23: renamed from R14; footprint (none) -> Resistor_SMD:R_0805_2012Metric
- R24: renamed from R15; footprint (none) -> Resistor_SMD:R_0805_2012Metric
- R29: renamed from R11; footprint (none) -> Resistor_SMD:R_0805_2012Metric
- SW1, SW2: footprint (none) -> Button_Switch_SMD:SW_SPST_PTS645Sx43SMTR92
- U7: footprint (none) -> Package_TO_SOT_SMD:SOT-223-3_TabPin2
- U8: footprint (none) -> PCM_Espressif:ESP32-WROOM-32E
- U9: footprint (none) -> Package_DFN_QFN:QFN-28-1EP_5x5mm_P0.5mm_EP3.35x3.35mm
- renumbered C1 to C18, C2 to C19, C6 to C21, C5 to C26, C3 to C5, C4 to C6, JP1 to JP9, R2 to R25, R7 to R26, R8 to R27, U2 to U10
Connections:
- net IO13 is gone; now on net MOSI_H: U8.16 (IO13)
- net +3V3: now also U5.1 (VDD)
- net GND: now also C14.1, C15.1, D5.2 (A), J1.2, U6.3 (GND), U6.5 (~{ON}/OFF)
- net MOSI_H: no longer R29.2, U8.37 (IO23)
- net VCC: no longer U5.1 (VDD)
- net Signal data DT11 renamed IO4
- new net: C14.2, J1.1, U6.1 (VIN)
- new net: D5.1 (K), L1.1, U6.2 (OUT)
- new net 5V regulated: C15.2, L1.2, U6.4 (FB)
- new net IO23: R29.2, U8.37 (IO23)
Other:
- note added: "9V Battery Input"

Commit message: Footprint Updates
Parts:
- removed I2C_PU0: S_MODE, KiCAD_Camsat_PCB:SMT-JUMPER_3_2-NC_TRACE_SILK, symbol KiCAD_Camsat_PCB-eagle-import:JUMPER-SMT_3_2-NC_TRACE_SILK
- removed LED0, SCX0, SDX0: JUMPER-SMT_2_NC_TRACE_SILK, KiCAD_Camsat_PCB:SMT-JUMPER_2_NC_TRACE_SILK, symbol KiCAD_Camsat_PCB-eagle-import:JUMPER-SMT_2_NC_TRACE_SILK
- added D6, D7: SS14, Diode_SMD:D_SMA, symbol Diode:SS14
- ADDR0: footprint KiCAD_Camsat_PCB:SMT-JUMPER_3_1-NC_TRACE_SILK -> Jumper:SolderJumper-2_P1.3mm_Bridged_Pad1.0x1.5mm
- C1, C18, C19, C2, C21, C26, C7: footprint e-radionica.com footprinti:0603C -> Capacitor_SMD:C_0603_1608Metric
- C3, C4: footprint KiCAD_Camsat_PCB:0805-NO -> Capacitor_SMD:C_0805_2012Metric
- C5, C6: footprint KiCAD_Camsat_PCB:0603 -> Capacitor_SMD:C_0603_1608Metric
- D1: footprint KiCAD_Camsat_PCB:LED-0603 -> LED_SMD:LED_0603_1608Metric
- D2: footprint KiCAD_Camsat_PCB:SOD-323 -> Diode_SMD:D_SOD-323
- J1: footprint (none) -> Connector_BarrelJack:BarrelJack_CUI_PJ-102AH_Horizontal
- JP1: footprint e-radionica.com footprinti:SMD_JUMPER -> Jumper:SolderJumper-2_P1.3mm_Open_Pad1.0x1.5mm
- JP9: footprint e-radionica.com footprinti:SMD-JUMPER-CONNECTED_TRACE_SLODERMASK -> Jumper:SolderJumper-2_P1.3mm_Bridged_Pad1.0x1.5mm
- K1: footprint e-radionica.com footprinti:HYC77-TF09-200 -> esp32:MICROSD-HYC77-TF09-200
- L1: footprint (none) -> Inductor_SMD:L_Bourns_SRN8040TA
- Q3, Q4: footprint KiCAD_Camsat_PCB:SOT23-WIDE -> Package_TO_SOT_SMD:SOT-23
- R1: footprint e-radionica.com footprinti:0603R -> Resistor_SMD:R_0805_2012Metric
- R2, R25, R3, R4, R5, R6: footprint KiCAD_Camsat_PCB:0603 -> Resistor_SMD:R_0805_2012Metric
- R26, R27, R7, R8: footprint KiCAD_Camsat_PCB:0805-NO -> Resistor_SMD:R_0805_2012Metric
- R9: footprint KiCAD_Camsat_PCB:_0805MP -> Resistor_SMD:R_0805_2012Metric
Connections:
- net PICO_AUX is gone; now on net GND: U1.P2 (SDX)
- net SCX is gone; now on net GND: U1.P3 (SCX)
- net +5V: now also D7.1 (K); no longer J4.2
- net 3.3V: now also R2.2, R25.2
- net GND: now also D1.C
- net at C14.2, U6.1 (VIN): now also D6.1 (K); no longer J1.1
- net 5V regulated renamed 5V Board
- new net: D6.2 (A), J1.1
- new net: D7.2 (A), J4.2
Other:
- note added: "SDA = GPIO21 SCL = GPIO22 CS = GPIO5 MOSI = GPIO13 SCLK = GPIO18 MISO = GPIO19"
- note removed: "0x6A"
- note removed: "0x6B"
- note removed: "Cut trace to disconnect Power LED."
- note removed: "GND"
- note removed: "OPEN"
- note removed: "SDA = GPIO21 SCL = GPIO22 CS = GPIO5 MOSI = GPIO23 SCLK = GPIO18 MISO = GPIO19"
- note removed: "SPI"
- note removed: "VDD"
- moved on the sheet: C14, J1

Commit message: All Footprints completed
Parts:
- U1: footprint KiCAD_Camsat_PCB:LGA-14L -> esp32:PQFN50P250X300X86-14N
- U10: footprint KiCAD_Camsat_PCB:BME280 -> esp32:PSON65P250X250X100-8N
- U2: footprint KiCAD_Camsat_PCB:SOT23-5 -> Package_TO_SOT_SMD:SOT-23-5
- U3: footprint e-radionica.com footprinti:SOT-23-5 -> Package_TO_SOT_SMD:SOT-23-5
Changed lines of the file:
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@@
 			)
 		)
-		(property "Footprint" "KiCAD_Camsat_PCB:LGA-14L"
+		(property "Footprint" "esp32:PQFN50P250X300X86-14N"
 			(at 370.84 124.46 0)
 			(effects
@@
 			)
 		)
-		(property "Footprint" "KiCAD_Camsat_PCB:BME280"
+		(property "Footprint" "esp32:PSON65P250X250X100-8N"
 			(at 664.21 200.66 0)
 			(effects
@@
 			)
 		)
-		(property "Footprint" "e-radionica.com footprinti:SOT-23-5"
+		(property "Footprint" "Package_TO_SOT_SMD:SOT-23-5"
 			(at 189.23 153.67 0)
 			(effects
@@
 			)
 		)
-		(property "Footprint" "KiCAD_Camsat_PCB:SOT23-5"
+		(property "Footprint" "Package_TO_SOT_SMD:SOT-23-5"
 			(at 806.45 124.46 0)
 			(effects

Commit message: schemaric errors
Parts:
- removed ADDR0: JUMPER-SMT_3_1-NC_TRACE_SILK, Jumper:SolderJumper-2_P1.3mm_Bridged_Pad1.0x1.5mm, symbol KiCAD_Camsat_PCB-eagle-import:JUMPER-SMT_3_1-NC_TRACE_SILK
- removed C2, C26: 2u2, Capacitor_SMD:C_0603_1608Metric, symbol e-radionica.com schematics:0603C
- removed C21, C7: 100n, Capacitor_SMD:C_0603_1608Metric, symbol e-radionica.com schematics:0603C
- removed C3, C4: 10uF, Capacitor_SMD:C_0805_2012Metric, symbol KiCAD_Camsat_PCB-eagle-import:microbuilder_CAP_CERAMIC0805-NOOUTLINE
- removed D2: 1N4148, Diode_SMD:D_SOD-323, symbol KiCAD_Camsat_PCB-eagle-import:microbuilder_DIODESOD-323
- removed JP1: SMD_JUMPER, Jumper:SolderJumper-2_P1.3mm_Open_Pad1.0x1.5mm, symbol e-radionica.com schematics:SMD_JUMPER
- removed JP9: SMD-JUMPER-CONNECTED_TRACE_SLODERMASK, Jumper:SolderJumper-2_P1.3mm_Bridged_Pad1.0x1.5mm, symbol e-radionica.com schematics:SMD-JUMPER-CONNECTED_TRACE_SLODERMASK
- removed Q3, Q4: BSS138, Package_TO_SOT_SMD:SOT-23, symbol KiCAD_Camsat_PCB-eagle-import:microbuilder_MOSFET-NWIDE
- removed R1: 10k, Resistor_SMD:R_0805_2012Metric, symbol e-radionica.com schematics:0603R
- removed R26, R27, R7, R8: 10K, Resistor_SMD:R_0805_2012Metric, symbol KiCAD_Camsat_PCB-eagle-import:microbuilder_RESISTOR0805_NOOUTLINE
- removed R5, R6: 10k, Resistor_SMD:R_0805_2012Metric, symbol KiCAD_Camsat_PCB-eagle-import:10KOHM-0603-1/10W-1%
- removed U2: MIC5225-3.3, Package_TO_SOT_SMD:SOT-23-5, symbol KiCAD_Camsat_PCB-eagle-import:microbuilder_VREG_SOT23-5
- removed U3: SE5218, Package_TO_SOT_SMD:SOT-23-5, symbol e-radionica.com schematics:SE5218
- removed U4: TXB0104QPWRQ1, e-radionica.com footprinti:TXB0104QPWRQ1, symbol e-radionica.com schematics:TXB0104QPWRQ1
- added C37: 100nF, Adafruit BMP280 (1):0805-NO, symbol Adafruit BMP280 (1)-eagle-import:CAP_CERAMIC0805-NOOUTLINE
- added D8: SS14, Diode_SMD:D_SMA, symbol Diode:SS14
- added R39: 10K, Resistor_SMD:R_0805_2012Metric, symbol KiCAD_Camsat_PCB-eagle-import:microbuilder_RESISTOR_0805MP
- J3: footprint Connector_USB:USB_Micro-B_Molex-105017-0001 -> esp32:MOLEX_105017-0001
Connections:
- net 3V3 is gone; now on net +3V3: C1.2, C18.2, C19.2, K1.4 (VDD)
- net CS_L is gone; now on net IO5: K1.2 (CS)
- net MOSI_H is gone; now on net IO13: U8.16 (IO13)
- net MOSI_L is gone; now on net IO13: K1.3 (MOSI)
- net SCK_3V is gone; now on net IO22: U10.4 (SCK)
- net SCLK_L is gone; now on net IO18: K1.5 (SCLK)
- net SDI_3V is gone; now on net IO21: U10.3 (SDI)
- net +5V: no longer C10.1, U7.3 (VIN)
- net +5V_VBUS: now also D8.2 (A)
- net 3.3V: now also U1.5 (VDD_IO), U1.8 (VDD), C37.1, R39.2; no longer U1.P5 (VDD_IO), U1.P8 (VDD)
- net CS_3V: now also R39.1
- net GND: now also J3.P$10 (EP), J3.P$6 (EP), J3.P$7 (EP), J3.P$8 (EP), J3.P$9 (EP), U1.1 (SDO/SA0), U1.2 (SDX), U1.3 (SCX), U1.6 (GND@6), U1.7 (GND@7), C37.2; no longer J3.10 (EP), J3.6 (EP), J3.7 (EP), J3.8 (EP), J3.9 (EP), U1.P2 (SDX), U1.P3 (SCX), U1.P6 (GND@6), U1.P7 (GND@7)
- net INT1: now also U1.4 (INT1); no longer U1.P4 (INT1)
- net IO21: now also U1.14 (SDA); no longer U1.P14 (SDA)
- net IO22: now also U1.13 (SCL); no longer U1.P13 (SCL)
- net OCS: now also U1.10 (OCS_AUX); no longer U1.P10 (OCS_AUX)
- net POCI_AUX: now also U1.11 (SDO_AUX); no longer U1.P11 (SDO_AUX)
- net ~{CS}: now also U1.12 (~{CS}); no longer U1.P12 (~{CS})
- net at R4.1: now also D1.1 (A); no longer D1.A
- net CS_H renamed IO5
- net MISO_H renamed IO19
- net MISO_L renamed IO13
- removed net POCI/SA0: U1.P1 (SDO/SA0)
- net SCLK_H renamed IO18
- new net 5V_Board: C10.1, D8.1 (K), U7.3 (VIN)
- no-connect marks 24 -> 27
Other:
- note added: "Maybe can be removed"
- note removed: "VOLTAGE LEVEL TRANSLATOR"
- note removed: "VOLTAGE REGULATOR"

Commit message: Power selection
Parts:
- removed D7: SS14, Diode_SMD:D_SMA, symbol Diode:SS14
- removed J4: 210-1S-1*3Ppin Gold-plated, Connector_PinHeader_2.54mm:PinHeader_1x03_P2.54mm_Vertical, symbol 210-1S-1*3Ppin Gold-plated
- C37: footprint Adafruit BMP280 (1):0805-NO -> Capacitor_SMD:C_0603_1608Metric
Other:
- note removed: "Maybe can be removed"

Commit message: Schematic Ready
Connections:
- net +3V3: no longer U7.4 (TAB)
- net EN: no longer SW1.2
- net GND: now also D1.2 (C), J3.P$1 (EP), J3.P$11 (EP), J3.P$12 (EP), J3.P$13 (EP), J3.P$2 (EP), K1.SHIELD (SH), SW1.2 (4), SW2.2 (4); no longer D1.C, J3.P$6 (EP), J3.P$7 (EP), SW1.3, SW1.4, SW2.3, SW2.4
- net INT2: now also U1.9 (INT2); no longer U1.P9 (INT2)
- net IO0_BTN: no longer SW2.2
- no-connect marks 27 -> 28
Other:
- moved on the sheet: C1, C18, C19, C37, C5, C6, D1, R10, R2, R25, R3, R39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
