File: KiCAD_Camsat_PCB/KiCAD_Camsat_PCB.kicad_sch (KiCad schematic)
At the start: 67 parts, among them J1 Barrel_Jack, J3 105017-0001, J5 DZ127R-11-02-25, K1 HYC77-TF09-200, Q1 2N7002T-7-F, Q2 SS8050-G_C164885, Q8 2N7002T-7-F, Q9 SS8050-G_C164885, SW1 PTS645SH50SMTR92LFS, SW2 PTS645SH50SMTR92LFS, U1 ISM330DHCX, U10 BME280, U5 DHT11, U6 LM2596S-5, U7 AMS1117-3.3_C347222, U8 ESP32-WROOM-32E(8MB), U9 CP2102N-A02-GQFN28R

Commit message: new changes
Parts:
- removed R19: 0Ω, Resistor_SMD:R_0805_2012Metric, symbol 0402WGF0000TCE
- removed R20: 0Ω, Resistor_SMD:R_0805_2012Metric, symbol 0402WGF0000TCE_1
Connections:
- net 3.3V is gone; now on net +3V3: C37.1, C5.1, C6.1, R2.2, R25.2, R3.2, R39.2, R4.2, R9.2, U1.5 (VDD_IO), U1.8 (VDD), U10.6 (VDDIO), U10.8 (VDD)
- net TXD is gone; now on net RXD0: U9.26 (TXD)
- net TXD0 is gone; now on net RXD: U8.35 (TXD0)

Commit message: Layout Revision
Removed unnecessary nets.
Added nets for copper pours.
Removed some non-critical components from schematic.
Still needs some extra vias and adjusting silkscreen.
Parts:
- removed C25: 100nF, Capacitor_SMD:C_0603_1608Metric, symbol CL05B104KO5NNNC_8
- removed D1: RED, LED_SMD:LED_0603_1608Metric, symbol KiCAD_Camsat_PCB-eagle-import:LED-RED0603
- removed J5: DZ127R-11-02-25, Connector_PinHeader_1.27mm:PinHeader_1x02_P1.27mm_Vertical, symbol DZ127R-11-02-25
- removed Q1: 2N7002T-7-F, Package_TO_SOT_SMD:SOT-523, symbol 2N7002T-7-F_1
- removed Q8: 2N7002T-7-F, Package_TO_SOT_SMD:SOT-523, symbol 2N7002T-7-F
- removed R14: 22Ω, Resistor_SMD:R_0805_2012Metric, symbol 0402WGF220JTCE
- removed R21: 10kΩ, Resistor_SMD:R_0805_2012Metric, symbol 0402WGF1002TCE_4
- removed R29: 1kΩ, Resistor_SMD:R_0805_2012Metric, symbol 0402WGF1001TCE_1
- removed R4: 1k, Resistor_SMD:R_0805_2012Metric, symbol KiCAD_Camsat_PCB-eagle-import:1KOHM-0603-1/10W-1%
- added H1, H2, H3, H4: MountingHole, MountingHole:MountingHole_2.5mm, symbol Mechanical:MountingHole
- added LED3: 0805G (Green), LED_SMD:LED_0805_2012Metric, symbol 0805G (Green)
- added R1: 5.1kΩ, Resistor_SMD:R_0805_2012Metric, symbol 0402WGF5101TCE
Connections:
- net 5V Board is gone; now on net 5V_Board: C15.2, L1.2, U6.4 (FB)
- net 5V_Board: now also R1.2
- net GND: now also LED3.2 (K)
- net 9VIN: now reaches C14.2, D6.1 (K), U6.1 (VIN)
- net 5V_out: now reaches D5.1 (K), L1.1, U6.2 (OUT)
- net 9V: now reaches D6.2 (A), J1.1
- net I34: no longer names the net of U8.6 (IO34)
- net I35: no longer names the net of U8.7 (IO35)
- net I36: no longer names the net of U8.4 (SENSOR_VP)
- net I39: no longer names the net of U8.5 (SENSOR_VN)
- net IO12: no longer names the net of U8.14 (IO12)
- net IO14: no longer names the net of U8.13 (IO14)
- net IO15: no longer names the net of U8.23 (IO15)
- net IO16: no longer names the net of U8.27 (IO16)
- net IO17: no longer names the net of U8.28 (IO17)
- net IO19: no longer names the net of U8.31 (IO19)
- net IO2: no longer names the net of U8.24 (IO2)
- net IO23: no longer names the net of U8.37 (IO23)
- net IO25: no longer names the net of U8.10 (IO25)
- net IO26: no longer names the net of U8.11 (IO26)
- net IO27: no longer names the net of U8.12 (IO27)
- net IO32: no longer names the net of U8.8 (IO32)
- net IO33: no longer names the net of U8.9 (IO33)
- net OCS: no longer names the net of U1.10 (OCS_AUX)
- new net: LED3.1 (A), R1.1
Other:
- note removed: "POWER INPUT SELECTION"
- moved on the sheet: C1, C10, C11, C12, C13, C14, C15, C16, C17, C18, C19, C20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

Commit message: Mounting Hole Size Changes
Parts:
- H1, H2, H3, H4: footprint MountingHole:MountingHole_2.5mm -> MountingHole:MountingHole_3mm
Changed lines of the file:
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@@
 			)
 		)
-		(property "Footprint" "MountingHole:MountingHole_2.5mm"
+		(property "Footprint" "MountingHole:MountingHole_3mm"
 			(at 450.85 67.31 0)
 			(effects
@@
 			)
 		)
-		(property "Footprint" "MountingHole:MountingHole_2.5mm"
+		(property "Footprint" "MountingHole:MountingHole_3mm"
 			(at 450.85 60.96 0)
 			(effects
@@
 			)
 		)
-		(property "Footprint" "MountingHole:MountingHole_2.5mm"
+		(property "Footprint" "MountingHole:MountingHole_3mm"
 			(at 450.85 54.61 0)
 			(effects
@@
 			)
 		)
-		(property "Footprint" "MountingHole:MountingHole_2.5mm"
+		(property "Footprint" "MountingHole:MountingHole_3mm"
 			(at 450.85 73.66 0)
 			(effects
