File: KiCAD_Camsat_PCB/_autosave-KiCAD_Camsat_PCB.kicad_pcb (KiCad board)
At the start: 2 copper layers, 92 parts, among them J1 Barrel_Jack, J3 105017-0001, J4 210-1S-1*3Ppin Gold-plated, J5 DZ127R-11-02-25, K1 HYC77-TF09-200, Q1 2N7002T-7-F, Q2 SS8050-G_C164885, Q3 BSS138, Q4 BSS138, Q8 2N7002T-7-F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

Commit message: Schematic Ready
Connections:
- D1 pad 2: (no net) -> GND
- J3 pad P$1: (no net) -> GND
- J3 pad P$11: (no net) -> GND
- J3 pad P$12: (no net) -> GND
- J3 pad P$13: (no net) -> GND
- J3 pad P$2: (no net) -> GND
- K1 pad SHIELD: (no net) -> GND
- U1 pad 9: (no net) -> /INT2
Changed lines of the file:
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@@
 	(net 110 "/IO5")
 	(net 111 "/IO19")
+	(net 112 "/INT2")
 	(footprint "Package_TO_SOT_SMD:SOT-23-5"
 		(layer "F.Cu")
@@
 			(roundrect_rratio 0.25)
 			(net 5 "+3V3")
-			(pinfunction "VOUT(TAB)")
+			(pinfunction "TAB")
 			(pintype "unspecified")
 		)
@@
 			(roundrect_rratio 0.25)
 			(net 5 "+3V3")
-			(pinfunction "VOUT(TAB)")
+			(pinfunction "TAB")
 			(pintype "unspecified")
 		)
@@
 			(size 1.2 1.5)
 			(layers "F.Cu" "F.Mask" "F.Paste")
+			(net 1 "GND")
+			(pinfunction "SH")
+			(pintype "bidirectional")
 		)
 		(pad "SHIELD" smd rect
@@
 			(size 1.2 2.2)
 			(layers "F.Cu" "F.Mask" "F.Paste")
+			(net 1 "GND")
+			(pinfunction "SH")
+			(pintype "bidirectional")
 		)
 		(pad "SHIELD" smd rect
@@
 			(size 1.6 1.5)
 			(layers "F.Cu" "F.Mask" "F.Paste")
+			(net 1 "GND")
+			(pinfunction "SH")
+			(pintype "bidirectional")
 		)
 		(pad "SHIELD" smd rect
@@
 			(size 1.2 2.2)
 			(layers "F.Cu" "F.Mask" "F.Paste")
+			(net 1 "GND")
+			(pinfunction "SH")
+			(pintype "bidirectional")
 		)
 		(embedded_fonts no)
@@
 			(layers "F.Cu" "F.Mask" "F.Paste")
 			(roundrect_rratio 0.25)
+			(net 1 "GND")
+			(pinfunction "C")
+			(pintype "passive")
 		)
 		(embedded_fonts no)
@@
 			(size 0.61 0.35)
 			(layers "F.Cu" "F.Paste")
+			(net 112 "/INT2")
+			(pinfunction "INT2")
+			(pintype "bidirectional")
 		)
 		(pad "10" smd rect
@@
 			(roundrect_rratio 0.1923076923)
 			(net 1 "GND")
-			(pinfunction "4")
+			(pinfunction "3")
 			(pintype "unspecified")
 		)
@@
 			(roundrect_rratio 0.1923076923)
 			(net 1 "GND")
-			(pinfunction "4")
+			(pinfunction "3")
 			(pintype "unspecified")
 		)
@@
 			(layers "*.Cu" "*.Mask")
 			(remove_unused_layers no)
+			(net 1 "GND")
+			(pinfunction "EP")
+			(pintype "unspecified")
 			(solder_mask_margin 0.0762)
 		)
@@
 			(layers "*.Cu" "*.Mask")
 			(remove_unused_layers no)
+			(net 1 "GND")
+			(pinfunction "EP")
+			(pintype "unspecified")
 			(solder_mask_margin 0.0762)
 		)
@@
 			(size 1.8 1.9)
 			(layers "F.Cu" "F.Mask" "F.Paste")
+			(net 1 "GND")
+			(pinfunction "EP")
+			(pintype "unspecified")
 			(solder_mask_margin 0.0762)
 		)
@@
 			(layers "*.Cu" "*.Mask")
 			(remove_unused_layers no)
+			(net 1 "GND")
+			(pinfunction "EP")
+			(pintype "unspecified")
 			(solder_mask_margin 0.0762)
 		)
@@
 			(layers "*.Cu" "*.Mask")
 			(remove_unused_layers no)
+			(net 1 "GND")
+			(pinfunction "EP")
+			(pintype "unspecified")
 			(solder_mask_margin 0.0762)
 		)
